File: PCB/rpi.brd (EAGLE design)
At the start: 75 x 70 mm, 62 parts, among them IC2 MC1541TO, IC4 MEGA16-A, X1 2526-

Commit message: On branch master 	modified:   PCB/eagle.epf 	modified:   PCB/rpi.brd 	modified:   PCB/rpi.sch 	modified:   RaspberryPI/RaspberryPI.pro.user
Parts:
- removed U$15, U$17: BAS0KFILM, tablet:SOD-523
- added C14: UWX0J101MCL1GB, tablet:UWX0J101MCL1GB
- added D1, D2: (no value), diode:MINIMELF
- moved U$5 1.57 mm to (51.6, 33.4)
Connections:
- net +5V: now also C14.+
- net GND: now also C14.-
- net N$19: now also D1.A; no longer U$17.A
- net N$3: now also D2.A; no longer U$15.A
- net PC3: now also D1.C, D2.C; no longer U$15.K, U$17.K
Routing:
- net N$23: track 19.3 -> 26.8 mm
- net +5V: track 250.4 -> 257.4 mm
- net GND: track 357.8 -> 351.4 mm
- net PC3: track 74.5 -> 72.5 mm
- net PA3: track 66.6 -> 68.3 mm
- net N$3: track 1.20 -> 1.82 mm
