File: PCB/rpi.sch (EAGLE design)
At the start: 62 parts, among them IC2 MC1541TO, IC4 MEGA16-A, X1 2526-

Commit message: On branch master 	modified:   PCB/eagle.epf 	modified:   PCB/rpi.brd 	modified:   PCB/rpi.sch 	modified:   RaspberryPI/RaspberryPI.pro.user
Parts:
- removed U$15, U$17: BAS0KFILM, tablet:BAS0KFILM
- added C14: UWX0J101MCL1GB, tablet:UWX0J101MCL1GB
- added D1, D2: (no value), diode:DIODE-MINIMELF
Connections:
- net +5V: now also C14.+
- net GND: now also C14.-
- net N$19: now also D1.A; no longer U$17.A
- net N$3: now also D2.A; no longer U$15.A
- net PC3: now also D1.C, D2.C; no longer U$15.K, U$17.K
Changed lines of the file:
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@@
 <part name="R15" library="rcl" deviceset="R-EU_" device="R1206"/>
 <part name="GND6" library="supply1" deviceset="GND" device=""/>
-<part name="U$15" library="tablet" deviceset="BAS0KFILM" device=""/>
-<part name="U$17" library="tablet" deviceset="BAS0KFILM" device=""/>
+<part name="D1" library="diode" deviceset="DIODE-" device="MINIMELF"/>
+<part name="D2" library="diode" deviceset="DIODE-" device="MINIMELF"/>
+<part name="C14" library="tablet" deviceset="UWX0J101MCL1GB" device=""/>
 </parts>
 <sheets>
@@
 <instance part="U$5" gate="G$1" x="317.5" y="223.52"/>
 <instance part="C6" gate="G$1" x="358.14" y="203.2"/>
-<instance part="C7" gate="G$1" x="351.79" y="203.2"/>
+<instance part="C7" gate="G$1" x="340.36" y="203.2"/>
 <instance part="C8" gate="G$1" x="276.86" y="189.23"/>
 <instance part="C9" gate="G$1" x="270.51" y="189.23"/>
@@
 <instance part="R15" gate="G$1" x="149.86" y="180.34"/>
 <instance part="GND6" gate="1" x="142.24" y="170.18"/>
-<instance part="U$15" gate="G$1" x="160.02" y="99.06"/>
-<instance part="U$17" gate="G$1" x="165.1" y="96.52"/>
+<instance part="D1" gate="G$1" x="165.1" y="96.52"/>
+<instance part="D2" gate="G$1" x="160.02" y="99.06"/>
+<instance part="C14" gate="G$1" x="350.52" y="203.2"/>
 </instances>
 <busses>
@@
 <junction x="304.8" y="167.64"/>
 <junction x="309.88" y="167.64"/>
-<pinref part="C7" gate="G$1" pin="-"/>
-<wire x1="351.79" y1="167.64" x2="345.44" y2="167.64" width="0.1524" layer="91"/>
-<wire x1="345.44" y1="167.64" x2="314.96" y2="167.64" width="0.1524" layer="91"/>
-<wire x1="351.79" y1="200.66" x2="351.79" y2="167.64" width="0.1524" layer="91"/>
+<wire x1="345.44" y1="167.64" x2="340.36" y2="167.64" width="0.1524" layer="91"/>
 <junction x="314.96" y="167.64"/>
 <pinref part="C8" gate="G$1" pin="2"/>
+<wire x1="340.36" y1="167.64" x2="314.96" y2="167.64" width="0.1524" layer="91"/>
 <wire x1="276.86" y1="184.15" x2="276.86" y2="167.64" width="0.1524" layer="91"/>
 <junction x="276.86" y="167.64"/>
@@
 <pinref part="C6" gate="G$1" pin="-"/>
 <wire x1="358.14" y1="200.66" x2="358.14" y2="167.64" width="0.1524" layer="91"/>
-<wire x1="358.14" y1="167.64" x2="351.79" y2="167.64" width="0.1524" layer="91"/>
-<junction x="351.79" y="167.64"/>
+<wire x1="358.14" y1="167.64" x2="350.52" y2="167.64" width="0.1524" layer="91"/>
 <pinref part="GND3" gate="1" pin="GND"/>
+<wire x1="350.52" y1="167.64" x2="345.44" y2="167.64" width="0.1524" layer="91"/>
 <wire x1="309.88" y1="165.1" x2="309.88" y2="167.64" width="0.1524" layer="91"/>
 <pinref part="R9" gate="G$1" pin="1"/>
@@
 <wire x1="259.08" y1="205.74" x2="259.08" y2="195.58" width="0.1524" layer="91"/>
 <junction x="259.08" y="195.58"/>
+<pinref part="C14" gate="G$1" pin="-"/>
+<wire x1="350.52" y1="200.66" x2="350.52" y2="167.64" width="0.1524" layer="91"/>
+<pinref part="C7" gate="G$1" pin="-"/>
+<wire x1="340.36" y1="200.66" x2="340.36" y2="167.64" width="0.1524" layer="91"/>
+<junction x="340.36" y="167.64"/>
+<junction x="350.52" y="167.64"/>
 </segment>
 <segment>
@@
 <wire x1="358.14" y1="210.82" x2="358.14" y2="213.36" width="0.1524" layer="91"/>
 <wire x1="358.14" y1="213.36" x2="358.14" y2="219.71" width="0.1524" layer="91"/>
-<wire x1="345.44" y1="210.82" x2="304.8" y2="210.82" width="0.1524" layer="91"/>
 <pinref part="C10" gate="G$1" pin="1"/>
+<wire x1="345.44" y1="210.82" x2="340.36" y2="210.82" width="0.1524" layer="91"/>
+<wire x1="340.36" y1="210.82" x2="304.8" y2="210.82" width="0.1524" layer="91"/>
 <wire x1="304.8" y1="210.82" x2="292.1" y2="210.82" width="0.1524" layer="91"/>
 <wire x1="345.44" y1="208.28" x2="345.44" y2="210.82" width="0.1524" layer="91"/>
-<wire x1="345.44" y1="210.82" x2="351.79" y2="210.82" width="0.1524" layer="91"/>
-<pinref part="C7" gate="G$1" pin="+"/>
-<wire x1="351.79" y1="210.82" x2="358.14" y2="210.82" width="0.1524" layer="91"/>
-<wire x1="351.79" y1="208.28" x2="351.79" y2="210.82" width="0.1524" layer="91"/>
+<wire x1="345.44" y1="210.82" x2="350.52" y2="210.82" width="0.1524" layer="91"/>
 <junction x="345.44" y="210.82"/>
-<junction x="351.79" y="210.82"/>
 <junction x="358.14" y="210.82"/>
 <pinref part="U$4" gate="G$1" pin="K"/>
+<wire x1="350.52" y1="210.82" x2="358.14" y2="210.82" width="0.1524" layer="91"/>
 <wire x1="347.98" y1="213.36" x2="351.79" y2="213.36" width="0.1524" layer="91"/>
 <junction x="358.14" y="213.36"/>
@@
 <junction x="304.8" y="200.66"/>
 <junction x="304.8" y="210.82"/>
+<pinref part="C14" gate="G$1" pin="+"/>
+<wire x1="350.52" y1="208.28" x2="350.52" y2="210.82" width="0.1524" layer="91"/>
+<pinref part="C7" gate="G$1" pin="+"/>
+<wire x1="340.36" y1="208.28" x2="340.36" y2="210.82" width="0.1524" layer="91"/>
+<junction x="350.52" y="210.82"/>
+<junction x="340.36" y="210.82"/>
 </segment>
 <segment>
@@
 <wire x1="182.88" y1="99.06" x2="182.88" y2="144.78" width="0.1524" layer="91"/>
 <pinref part="U$1" gate="G$1" pin="S/S"/>
-<wire x1="165.1" y1="99.06" x2="182.88" y2="99.06" width="0.1524" layer="91"/>
+<wire x1="162.56" y1="99.06" x2="182.88" y2="99.06" width="0.1524" layer="91"/>
 <wire x1="233.68" y1="203.2" x2="276.86" y2="203.2" width="0.1524" layer="91"/>
-<pinref part="U$15" gate="G$1" pin="K"/>
-<pinref part="U$17" gate="G$1" pin="K"/>
 <wire x1="276.86" y1="203.2" x2="281.94" y2="203.2" width="0.1524" layer="91"/>
-<wire x1="170.18" y1="96.52" x2="182.88" y2="96.52" width="0.1524" layer="91"/>
+<wire x1="167.64" y1="96.52" x2="182.88" y2="96.52" width="0.1524" layer="91"/>
 <wire x1="182.88" y1="96.52" x2="182.88" y2="99.06" width="0.1524" layer="91"/>
 <junction x="182.88" y="99.06"/>
@@
 <wire x1="276.86" y1="205.74" x2="276.86" y2="203.2" width="0.1524" layer="91"/>
 <junction x="276.86" y="203.2"/>
+<pinref part="D2" gate="G$1" pin="C"/>
+<pinref part="D1" gate="G$1" pin="C"/>
 </segment>
 </net>
@@
 <wire x1="157.48" y1="40.64" x2="157.48" y2="96.52" width="0.1524" layer="91"/>
 <wire x1="157.48" y1="96.52" x2="147.32" y2="96.52" width="0.1524" layer="91"/>
-<pinref part="U$17" gate="G$1" pin="A"/>
-<wire x1="160.02" y1="96.52" x2="157.48" y2="96.52" width="0.1524" layer="91"/>
 <junction x="157.48" y="96.52"/>
+<pinref part="D1" gate="G$1" pin="A"/>
+<wire x1="162.56" y1="96.52" x2="157.48" y2="96.52" width="0.1524" layer="91"/>
 </segment>
 </net>
@@
 <segment>
 <pinref part="IC4" gate="G$1" pin="(TMS)PC3"/>
-<pinref part="U$15" gate="G$1" pin="A"/>
-<wire x1="147.32" y1="99.06" x2="154.94" y2="99.06" width="0.1524" layer="91"/>
-</segment>
-</net>
+<wire x1="147.32" y1="99.06" x2="157.48" y2="99.06" width="0.1524" layer="91"/>
+<pinref part="D2" gate="G$1" pin="A"/>
+</segment>
+</net>

Commit message: On branch master 	modified:   PCB/eagle.epf 	modified:   PCB/rpi.brd 	modified:   PCB/rpi.sch 	modified:   RaspberryPI/mainwindow.cpp 	modified:   RaspberryPI/mainwindow.h 	modified:   RaspberryPI/mainwindow.ui
Parts:
- U$14, U$2: device NX7002AK:NX7002AK -> tablet:NX7002AK
- U$8: device max1811:MAX1811 -> tablet:MAX1811
Connections:
- removed net N$24: SV1.6, X1-19.KL
- removed net N$27: SV1.8, X1-24.KL
- new net N$21: SV1.5, X1-19.KL
- new net N$22: SV1.1, X1-23.KL
- net N$4: now also SV1.3; no longer SV1.4
- net N$5: now also SV1.7, X1-24.KL; no longer SV1.2, X1-23.KL
- net PB4: now also SV1.8; no longer SV1.7
- net PB5: now also SV1.6; no longer SV1.5
- net PB6: now also SV1.4; no longer SV1.3
- net SCK: now also SV1.2; no longer SV1.1
Changed lines of the file:
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@@
 <grid distance="0.1" unitdist="inch" unit="inch" style="lines" multiple="1" display="no" altdistance="0.01" altunitdist="inch" altunit="inch"/>
 <layers>
-<layer number="1" name="Top" color="4" fill="1" visible="no" active="no"/>
-<layer number="16" name="Bottom" color="1" fill="1" visible="no" active="no"/>
-<layer number="17" name="Pads" color="2" fill="1" visible="no" active="no"/>
-<layer number="18" name="Vias" color="2" fill="1" visible="no" active="no"/>
-<layer number="19" name="Unrouted" color="6" fill="1" visible="no" active="no"/>
-<layer number="20" name="Dimension" color="15" fill="1" visible="no" active="no"/>
-<layer number="21" name="tPlace" color="7" fill="1" visible="no" active="no"/>
-<layer number="22" name="bPlace" color="7" fill="1" visible="no" active="no"/>
-<layer number="23" name="tOrigins" color="15" fill="1" visible="no" active="no"/>
-<layer number="24" name="bOrigins" color="15" fill="1" visible="no" active="no"/>
-<layer number="25" name="tNames" color="7" fill="1" visible="no" active="no"/>
-<layer number="26" name="bNames" color="7" fill="1" visible="no" active="no"/>
-<layer number="27" name="tValues" color="7" fill="1" visible="no" active="no"/>
-<layer number="28" name="bValues" color="7" fill="1" visible="no" active="no"/>
+<layer number="1" name="Top" color="4" fill="1" visible="yes" active="no"/>
+<layer number="16" name="Bottom" color="1" fill="1" visible="yes" active="no"/>
+<layer number="17" name="Pads" color="2" fill="1" visible="yes" active="no"/>
+<layer number="18" name="Vias" color="2" fill="1" visible="yes" active="no"/>
+<layer number="19" name="Unrouted" color="6" fill="1" visible="yes" active="no"/>
+<layer number="20" name="Dimension" color="15" fill="1" visible="yes" active="no"/>
+<layer number="21" name="tPlace" color="7" fill="1" visible="yes" active="no"/>
+<layer number="22" name="bPlace" color="7" fill="1" visible="yes" active="no"/>
+<layer number="23" name="tOrigins" color="15" fill="1" visible="yes" active="no"/>
+<layer number="24" name="bOrigins" color="15" fill="1" visible="yes" active="no"/>
+<layer number="25" name="tNames" color="7" fill="1" visible="yes" active="no"/>
+<layer number="26" name="bNames" color="7" fill="1" visible="yes" active="no"/>
+<layer number="27" name="tValues" color="7" fill="1" visible="yes" active="no"/>
+<layer number="28" name="bValues" color="7" fill="1" visible="yes" active="no"/>
 <layer number="29" name="tStop" color="7" fill="3" visible="no" active="no"/>
 <layer number="30" name="bStop" color="7" fill="6" visible="no" active="no"/>
@@
 <layer number="35" name="tGlue" color="7" fill="4" visible="no" active="no"/>
 <layer number="36" name="bGlue" color="7" fill="5" visible="no" active="no"/>
-<layer number="37" name="tTest" color="7" fill="1" visible="no" active="no"/>
-<layer number="38" name="bTest" color="7" fill="1" visible="no" active="no"/>
+<layer number="37" name="tTest" color="7" fill="1" visible="yes" active="no"/>
+<layer number="38" name="bTest" color="7" fill="1" visible="yes" active="no"/>
 <layer number="39" name="tKeepout" color="4" fill="11" visible="no" active="no"/>
 <layer number="40" name="bKeepout" color="1" fill="11" visible="no" active="no"/>
@@
 <layer number="44" name="Drills" color="7" fill="1" visible="no" active="no"/>
 <layer number="45" name="Holes" color="7" fill="1" visible="no" active="no"/>
-<layer number="46" name="Milling" color="3" fill="1" visible="no" active="no"/>
-<layer number="47" name="Measures" color="7" fill="1" visible="no" active="no"/>
-<layer number="48" name="Document" color="7" fill="1" visible="no" active="no"/>
-<layer number="49" name="Reference" color="7" fill="1" visible="no" active="no"/>
-<layer number="51" name="tDocu" color="6" fill="9" visible="no" active="no"/>
-<layer number="52" name="bDocu" color="7" fill="1" visible="no" active="no"/>
+<layer number="46" name="Milling" color="3" fill="1" visible="yes" active="no"/>
+<layer number="47" name="Measures" color="7" fill="1" visible="yes" active="no"/>
+<layer number="48" name="Document" color="7" fill="1" visible="yes" active="no"/>
+<layer number="49" name="Reference" color="7" fill="1" visible="yes" active="no"/>
+<layer number="51" name="tDocu" color="7" fill="1" visible="yes" active="no"/>
+<layer number="52" name="bDocu" color="7" fill="1" visible="yes" active="no"/>
 <layer number="91" name="Nets" color="2" fill="1" visible="yes" active="yes"/>
 <layer number="92" name="Busses" color="1" fill="1" visible="yes" active="yes"/>
@@
 <part name="X1" library="con-3m" deviceset="2526-" device=""/>
 <part name="SV1" library="con-lstb" deviceset="MA04-2" device=""/>
-<part name="U$2" library="NX7002AK" deviceset="NX7002AK" device=""/>
-<part name="U$8" library="max1811" deviceset="MAX1811" device=""/>
+<part name="U$2" library="tablet" deviceset="NX7002AK" device=""/>
+<part name="U$8" library="tablet" deviceset="MAX1811" device=""/>
 <part name="U$1" library="tablet" deviceset="LT1619" device="S"/>
 <part name="C1" library="rcl" deviceset="C-EU" device="C1206"/>
@@
 <part name="P+3" library="supply1" deviceset="+5V" device=""/>
 <part name="JP6" library="pinhead" deviceset="PINHD-1X1" device=""/>
-<part name="U$14" library="NX7002AK" deviceset="NX7002AK" device=""/>
+<part name="U$14" library="tablet" deviceset="NX7002AK" device=""/>
 <part name="GND5" library="supply1" deviceset="GND" device=""/>
 <part name="JP7" library="pinhead" deviceset="PINHD-1X1" device=""/>
@@
 <instance part="X1" gate="-25" x="236.22" y="33.02" rot="R180"/>
 <instance part="X1" gate="-26" x="332.74" y="40.64" rot="R180"/>
-<instance part="SV1" gate="G$1" x="210.82" y="111.76" rot="R180"/>
+<instance part="SV1" gate="G$1" x="210.82" y="111.76" rot="MR180"/>
 <instance part="U$2" gate="G$1" x="185.42" y="43.18" rot="MR270"/>
 <instance part="U$8" gate="G$1" x="208.28" y="198.12"/>
@@
 <net name="N$4" class="0">
 <segment>
-<pinref part="SV1" gate="G$1" pin="4"/>
-<wire x1="218.44" y1="114.3" x2="220.98" y2="114.3" width="0.1524" layer="91"/>
 <pinref part="R4" gate="G$1" pin="2"/>
 <wire x1="220.98" y1="83.82" x2="220.98" y2="114.3" width="0.1524" layer="91"/>
+<pinref part="SV1" gate="G$1" pin="3"/>
+<wire x1="218.44" y1="114.3" x2="220.98" y2="114.3" width="0.1524" layer="91"/>
 </segment>
 </net>
@@
 <wire x1="281.94" y1="198.12" x2="276.86" y2="198.12" width="0.1524" layer="91"/>
 <junction x="276.86" y="198.12"/>
-</segment>
-</net>
-<net name="N$5" class="0">
-<segment>
-<pinref part="X1" gate="-23" pin="KL"/>
-<pinref part="SV1" gate="G$1" pin="2"/>
-<wire x1="226.06" y1="116.84" x2="218.44" y2="116.84" width="0.1524" layer="91"/>
-</segment>
-</net>
-<net name="N$24" class="0">
-<segment>
-<pinref part="X1" gate="-19" pin="KL"/>
-<pinref part="SV1" gate="G$1" pin="6"/>
-<wire x1="226.06" y1="111.76" x2="218.44" y2="111.76" width="0.1524" layer="91"/>
-</segment>
-</net>
-<net name="N$27" class="0">
-<segment>
-<pinref part="SV1" gate="G$1" pin="8"/>
-<wire x1="218.44" y1="109.22" x2="226.06" y2="109.22" width="0.1524" layer="91"/>
-<pinref part="X1" gate="-24" pin="KL"/>
 </segment>
 </net>
@@
 <segment>
 <pinref part="IC4" gate="G$1" pin="(MISO)PB6"/>
-<pinref part="SV1" gate="G$1" pin="3"/>
-<wire x1="203.2" y1="114.3" x2="198.12" y2="114.3" width="0.1524" layer="91"/>
 <wire x1="198.12" y1="114.3" x2="198.12" y2="129.54" width="0.1524" layer="91"/>
 <pinref part="JP1" gate="1" pin="3"/>
@@
 <wire x1="147.32" y1="129.54" x2="198.12" y2="129.54" width="0.1524" layer="91"/>
 <junction x="198.12" y="129.54"/>
+<pinref part="SV1" gate="G$1" pin="4"/>
+<wire x1="203.2" y1="114.3" x2="198.12" y2="114.3" width="0.1524" layer="91"/>
 </segment>
 </net>
@@
 <segment>
 <pinref part="IC4" gate="G$1" pin="(MOSI)PB5"/>
-<pinref part="SV1" gate="G$1" pin="5"/>
-<wire x1="203.2" y1="111.76" x2="195.58" y2="111.76" width="0.1524" layer="91"/>
 <wire x1="195.58" y1="111.76" x2="195.58" y2="127" width="0.1524" layer="91"/>
 <pinref part="JP1" gate="1" pin="4"/>
@@
 <wire x1="147.32" y1="127" x2="195.58" y2="127" width="0.1524" layer="91"/>
 <junction x="195.58" y="127"/>
+<pinref part="SV1" gate="G$1" pin="6"/>
+<wire x1="203.2" y1="111.76" x2="195.58" y2="111.76" width="0.1524" layer="91"/>
 </segment>
 </net>
@@
 <segment>
 <pinref part="IC4" gate="G$1" pin="(SS)PB4"/>
-<pinref part="SV1" gate="G$1" pin="7"/>
-<wire x1="203.2" y1="109.22" x2="193.04" y2="109.22" width="0.1524" layer="91"/>
 <wire x1="193.04" y1="109.22" x2="193.04" y2="124.46" width="0.1524" layer="91"/>
 <wire x1="193.04" y1="124.46" x2="147.32" y2="124.46" width="0.1524" layer="91"/>
+<pinref part="SV1" gate="G$1" pin="8"/>
+<wire x1="203.2" y1="109.22" x2="193.04" y2="109.22" width="0.1524" layer="91"/>
 </segment>
 </net>
@@
 <net name="SCK" class="0">
 <segment>
-<pinref part="SV1" gate="G$1" pin="1"/>
-<wire x1="203.2" y1="116.84" x2="200.66" y2="116.84" width="0.1524" layer="91"/>
 <wire x1="200.66" y1="116.84" x2="200.66" y2="132.08" width="0.1524" layer="91"/>
 <pinref part="JP1" gate="1" pin="2"/>
@@
 <wire x1="147.32" y1="132.08" x2="200.66" y2="132.08" width="0.1524" layer="91"/>
 <junction x="200.66" y="132.08"/>
+<pinref part="SV1" gate="G$1" pin="2"/>
+<wire x1="203.2" y1="116.84" x2="200.66" y2="116.84" width="0.1524" layer="91"/>
 </segment>
 </net>
@@
 </segment>
 </net>
+<net name="N$5" class="0">
+<segment>
+<pinref part="SV1" gate="G$1" pin="7"/>
+<pinref part="X1" gate="-24" pin="KL"/>
+<wire x1="218.44" y1="109.22" x2="226.06" y2="109.22" width="0.1524" layer="91"/>
+</segment>
+</net>
+<net name="N$21" class="0">
+<segment>
+<pinref part="SV1" gate="G$1" pin="5"/>
+<pinref part="X1" gate="-19" pin="KL"/>
+<wire x1="218.44" y1="111.76" x2="226.06" y2="111.76" width="0.1524" layer="91"/>
+</segment>
+</net>
+<net name="N$22" class="0">
+<segment>
+<pinref part="SV1" gate="G$1" pin="1"/>
+<pinref part="X1" gate="-23" pin="KL"/>
+<wire x1="218.44" y1="116.84" x2="226.06" y2="116.84" width="0.1524" layer="91"/>
+</segment>
+</net>
